Commit message: 파일 분리
LiDAR, Camera, robot_core 파일 분리

File: src/forey_demo/description/robot.urdf.xacro (robot description, xacro)
@@ -2,3 +2,5 @@
 <robot xmlns:xacro="http://www.ros.org/wiki/xacro"  name="robot">
     <xacro:include filename="robot_core.xacro" />
+    <xacro:include filename="lidar.xacro" />
+    <xacro:include filename="camera.xacro" />
 </robot>

File: src/forey_demo/description/robot_core.xacro (robot description, xacro)
@@ -118,34 +118,3 @@
         </visual>
     </link>
-    <!-- LiDAR_LINK -->
-    <joint name="LiDAR_joint" type="fixed">
-        <parent link="chassis" />
-        <child link="laser_frame" />
-        <origin xyz="0.141188 0 ${0.1448+white_plate_thickness}" rpy="0 0 0" />
-    </joint>
-    <link name="laser_frame">
-        <visual>
-            <geometry>
-                <cylinder radius="0.0385" length="0.019" />
-            </geometry>
-            <material name="green" />
-        </visual>
-    </link>
-    <!-- CAMERA_LINK -->
-    <xacro:property name="camera_thickness" value="0.031" />
-    <xacro:property name="chassis_to_camera_x" value="${0.210658 + camera_plate_thickness + camera_thickness/2}" />
-    <xacro:property name="chassis_to_camera_z" value="0.0156962" />
-    <joint name="camera_joint" type="fixed">
-        <parent link="chassis" />
-        <child link="camera_link" />
-        <origin xyz="${chassis_to_camera_x} 0 ${chassis_to_camera_z+box_z}" rpy="0 0 0" />
-    </joint>©
-    <link name="camera_link">
-        <visual>
-            <geometry>
-                <box size="${camera_thickness} 0.09 0.022" />
-            </geometry>
-            <material name="red" />
-        </visual>
-    </link>
 </robot>
