Commit message: 샘플 수정 코드
샘플 수정 코드

File: src/forey_demo/description/robot_core.xacro (robot description, xacro)
@@ -85,8 +85,9 @@
         </visual>
     </link>
+    <!-- dasfsdf -->
     <!-- RIGHT_FRONT_WHEEL_LINK -->
     <joint name="right_front_wheel_joint" type="continuous">
         <parent link="chassis" />
-        <child link="right_front_wheel" />
+        <child link="right_front_wheel" />˝
         <origin xyz="${box_x/2+base_link_to_wheel_x} -${base_link_to_wheel_y+box_y/2} ${base_link_to_wheel_z}" rpy="-${pi/2} 0 0" />
         <axis xyz="0 0 1" />
@@ -100,4 +101,5 @@
         </visual>
     </link>
+©˝˝˝˝
     <!-- RIGHT_REAR_WHEEL_LINK -->
     <joint name="right_rear_wheel_joint" type="continuous">

Commit message: update urdf 작성
샤시와 바퀴 4개

라이다, 카메라

File: src/forey_demo/description/robot_core.xacro (robot description, xacro)
@@ -28,5 +28,5 @@
     <xacro:property name="box_x" value="0.203" />
     <xacro:property name="box_y" value="0.106" />
-    <xacro:property name="box_z" value="0.056" />
+    <xacro:property name="box_z" value="0.057" />
     <!-- BASE_FOOTPRINT: 지면 기준 고정 프레임 (내비게이션, TF 트리용) -->
     <link name="base_footprint" />
@@ -85,10 +85,9 @@
         </visual>
     </link>
-    <!-- dasfsdf -->
     <!-- RIGHT_FRONT_WHEEL_LINK -->
     <joint name="right_front_wheel_joint" type="continuous">
         <parent link="chassis" />
-        <child link="right_front_wheel" />˝
-        <origin xyz="${box_x/2+base_link_to_wheel_x} -${base_link_to_wheel_y+box_y/2} ${base_link_to_wheel_z}" rpy="-${pi/2} 0 0" />
+        <child link="right_front_wheel" />
+        <origin xyz="${box_x/2+base_link_to_wheel_x} -${base_link_to_wheel_y+box_y/2+wheel_width/2} ${base_link_to_wheel_z}" rpy="-${pi/2} 0 0" />
         <axis xyz="0 0 1" />
     </joint>
@@ -101,10 +100,9 @@
         </visual>
     </link>
-©˝˝˝˝
     <!-- RIGHT_REAR_WHEEL_LINK -->
     <joint name="right_rear_wheel_joint" type="continuous">
         <parent link="chassis" />
         <child link="right_rear_wheel" />
-        <origin xyz="${box_x/2-base_link_to_wheel_x} -${base_link_to_wheel_y+box_y/2} ${base_link_to_wheel_z}" rpy="-${pi/2} 0 0" />
+        <origin xyz="${box_x/2-base_link_to_wheel_x} -${base_link_to_wheel_y+box_y/2+wheel_width/2} ${base_link_to_wheel_z}" rpy="-${pi/2} 0 0" />
         <axis xyz="0 0 1" />
     </joint>

Commit message: 수정 코드
수정 코드

File: src/forey_demo/description/robot_core.xacro (robot description, xacro)
@@ -67,5 +67,5 @@
                 <cylinder radius="${wheel_radius}" length="${wheel_width}" />
             </geometry>
-            <material name="red" />
+            <material name="blue" />
         </visual>
     </link>
@@ -115,3 +115,17 @@
         </visual>
     </link>
+    <!-- LiDAR_LINK -->
+    <joint name="LiDAR_joint" type="fixed">
+        <parent link="chassis" />
+        <child link="laser_frame" />
+        <origin xyz="0.141188 0 0.1448" rpy="0 0 0" />
+    </joint>
+    <link name="laser_frame">
+        <visual>
+            <geometry>
+                <cylinder radius="0.0385" length="0.019" />
+            </geometry>
+            <material name="green" />
+        </visual>
+    </link>
 </robot>

Commit message: update LiDAR, Camera
라이다 화이트 플레이트 높이 적용
카메라 비주얼 작성

File: src/forey_demo/description/robot_core.xacro (robot description, xacro)
@@ -29,4 +29,7 @@
     <xacro:property name="box_y" value="0.106" />
     <xacro:property name="box_z" value="0.057" />
+    <xacro:property name="white_plate_thickness" value="0.002" />
+    <xacro:property name="green_plate_thickness" value="0.005" />
+    <xacro:property name="camera_plate_thickness" value="0.004" />
     <!-- BASE_FOOTPRINT: 지면 기준 고정 프레임 (내비게이션, TF 트리용) -->
     <link name="base_footprint" />
@@ -119,5 +122,5 @@
         <parent link="chassis" />
         <child link="laser_frame" />
-        <origin xyz="0.141188 0 0.1448" rpy="0 0 0" />
+        <origin xyz="0.141188 0 ${0.1448+white_plate_thickness}" rpy="0 0 0" />
     </joint>
     <link name="laser_frame">
@@ -129,3 +132,20 @@
         </visual>
     </link>
+    <!-- CAMERA_LINK -->
+    <xacro:property name="camera_thickness" value="0.031" />
+    <xacro:property name="chassis_to_camera_x" value="${0.210658 + camera_plate_thickness + camera_thickness/2}" />
+    <xacro:property name="chassis_to_camera_z" value="0.0156962" />
+    <joint name="camera_joint" type="fixed">
+        <parent link="chassis" />
+        <child link="camera_link" />
+        <origin xyz="${chassis_to_camera_x} 0 ${chassis_to_camera_z+box_z}" rpy="0 0 0" />
+    </joint>©
+    <link name="camera_link">
+        <visual>
+            <geometry>
+                <box size="${camera_thickness} 0.09 0.022" />
+            </geometry>
+            <material name="red" />
+        </visual>
+    </link>
 </robot>

Commit message: URDF 수정 코드2
URDF 수정 코드2

File: src/forey_demo/description/robot_core.xacro (robot description, xacro)
@@ -1,26 +1,13 @@
 <?xml version="1.0"?>
-<robot xmlns:xacro="http://www.ros.org/wiki/xacro"  name="robot">
+<robot xmlns:xacro="http://www.ros.org/wiki/xacro" name="robot">
     <xacro:property name="pi" value="3.14159265359" />
-    <material name="white">
-        <color rgba="1.0 1.0 1.0 1.0" />
-    </material>
-    <material name="orange">
-        <color rgba="1.0 0.5 0.0 1.0" />
-    </material>
-    <material name="blue">
-        <color rgba="0.0 0.0 1.0 1.0" />
-    </material>
-    <material name="green">
-        <color rgba="0.0 1.0 0.0 1.0" />
-    </material>
-    <material name="red">
-        <color rgba="1.0 0.0 0.0 1.0" />
-    </material>
-    <!-- 바퀴 치수 -->
+    <material name="white"><color rgba="1.0 1.0 1.0 1.0" /></material>
+    <material name="orange"><color rgba="1.0 0.5 0.0 1.0" /></material>
+    <material name="blue"><color rgba="0.0 0.0 1.0 1.0" /></material>
+    <material name="green"><color rgba="0.0 1.0 0.0 1.0" /></material>
+    <material name="red"><color rgba="1.0 0.0 0.0 1.0" /></material>
     <xacro:property name="wheel_diameter" value="0.0745" />
     <xacro:property name="wheel_radius" value="${wheel_diameter/2}" />
-    <!-- 바퀴 두께 -->
     <xacro:property name="wheel_width" value="0.02" />
-    <!-- base_link 기준 바퀴 위치 -->
     <xacro:property name="base_link_to_wheel_x" value="0.077" />
     <xacro:property name="base_link_to_wheel_y" value="0.0235" />
@@ -30,9 +17,23 @@
     <xacro:property name="box_z" value="0.057" />
     <xacro:property name="white_plate_thickness" value="0.002" />
-    <xacro:property name="green_plate_thickness" value="0.005" />
-    <xacro:property name="camera_plate_thickness" value="0.004" />
-    <!-- BASE_FOOTPRINT: 지면 기준 고정 프레임 (내비게이션, TF 트리용) -->
+    <xacro:macro name="inertial_box" params="mass x y z *origin">
+        <inertial>
+            <xacro:insert_block name="origin"/>
+            <mass value="${mass}" />
+            <inertia ixx="${(1/12) * mass * (y*y+z*z)}" ixy="0.0" ixz="0.0"
+                    iyy="${(1/12) * mass * (x*x+z*z)}" iyz="0.0"
+                    izz="${(1/12) * mass * (x*x+y*y)}" />
+        </inertial>
+    </xacro:macro>
+    <xacro:macro name="inertial_cylinder" params="mass radius length *origin">
+        <inertial>
+            <xacro:insert_block name="origin"/>
+            <mass value="${mass}" />
+            <inertia ixx="${(1/12) * mass * (3*radius*radius + length*length)}" ixy="0.0" ixz="0.0"
+                    iyy="${(1/12) * mass * (3*radius*radius + length*length)}" iyz="0.0"
+                    izz="${(1/2) * mass * (radius*radius)}" />
+        </inertial>
+    </xacro:macro>
     <link name="base_footprint" />
-    <!-- BASE_FOOTPRINT -> BASE_LINK: base_link는 바퀴 반지름(0.05)만큼 지면 위 -->
     <joint name="base_footprint_joint" type="fixed">
         <parent link="base_footprint" />
@@ -40,8 +41,5 @@
         <origin xyz="0 0 ${wheel_radius}" rpy="0 0 0" />
     </joint>
-    <!-- BASE_LINK -->
-    <link name="base_link">
-    </link>
-    <!-- CHASSIS_LINK -->
+    <link name="base_link" />
     <joint name="chassis_joint" type="fixed">
         <parent link="base_link" />
@@ -51,72 +49,44 @@
     <link name="chassis">
         <visual>
-            <origin xyz="${box_x/2} 0.0 ${box_z/2}" rpy="0 0 0" />
-            <geometry>
-                <box size="${box_x} ${box_y} ${box_z}" />
-            </geometry>
+            <origin xyz="${box_x/2} 0.0 ${box_z/2}" />
+            <geometry><box size="${box_x} ${box_y} ${box_z}" /></geometry>
             <material name="white" />
         </visual>
+        <collision>
+            <origin xyz="${box_x/2} 0.0 ${box_z/2}" />
+            <geometry><box size="${box_x} ${box_y} ${box_z}" /></geometry>
+        </collision>
+        <xacro:inertial_box mass="0.8" x="${box_x}" y="${box_y}" z="${box_z}">
+            <origin xyz="${box_x/2} 0.0 ${box_z/2}" rpy="0 0 0"/>
+        </xacro:inertial_box>
     </link>
-    <!-- LEFT_FRONT_WHEEL_LINK -->
-    <joint name="left_front_wheel_joint" type="continuous">
-        <parent link="chassis" />
-        <child link="left_front_wheel" />
-        <origin xyz="${base_link_to_wheel_x+box_x/2} ${base_link_to_wheel_y+box_y/2+wheel_width/2} ${base_link_to_wheel_z}" rpy="-${pi/2} 0 0" />
-        <axis xyz="0 0 1" />
-    </joint>
-    <link name="left_front_wheel">
-        <visual>
-            <geometry>
-                <cylinder radius="${wheel_radius}" length="${wheel_width}" />
-            </geometry>
-            <material name="blue" />
-        </visual>
-    </link>
-    <!-- LEFT_REAR_WHEEL_LINK -->
-    <joint name="left_rear_wheel_joint" type="continuous">
-        <parent link="chassis" />
-        <child link="left_rear_wheel" />
-        <origin xyz="${box_x/2-base_link_to_wheel_x} ${base_link_to_wheel_y+box_y/2+wheel_width/2} ${base_link_to_wheel_z}" rpy="-${pi/2} 0 0" />
-        <axis xyz="0 0 1" />
-    </joint>
-    <link name="left_rear_wheel">
-        <visual>
-            <geometry>
-                <cylinder radius="${wheel_radius}" length="${wheel_width}" />
-            </geometry>
-            <material name="blue" />
-        </visual>
-    </link>
-    <!-- RIGHT_FRONT_WHEEL_LINK -->
-    <joint name="right_front_wheel_joint" type="continuous">
-        <parent link="chassis" />
-        <child link="right_front_wheel" />
-        <origin xyz="${box_x/2+base_link_to_wheel_x} -${base_link_to_wheel_y+box_y/2+wheel_width/2} ${base_link_to_wheel_z}" rpy="-${pi/2} 0 0" />
-        <axis xyz="0 0 1" />
-    </joint>
-    <link name="right_front_wheel">
-        <visual>
-            <geometry>
-                <cylinder radius="${wheel_radius}" length="${wheel_width}" />
-            </geometry>
-            <material name="blue" />
-        </visual>
-    </link>
-    <!-- RIGHT_REAR_WHEEL_LINK -->
-    <joint name="right_rear_wheel_joint" type="continuous">
-        <parent link="chassis" />
-        <child link="right_rear_wheel" />
-        <origin xyz="${box_x/2-base_link_to_wheel_x} -${base_link_to_wheel_y+box_y/2+wheel_width/2} ${base_link_to_wheel_z}" rpy="-${pi/2} 0 0" />
-        <axis xyz="0 0 1" />
-    </joint>
-    <link name="right_rear_wheel">
-        <visual>
-            <geometry>
-                <cylinder radius="${wheel_radius}" length="${wheel_width}" />
-            </geometry>
-            <material name="blue" />
-        </visual>
-    </link>
-    <!-- LiDAR_LINK -->
+    <xacro:macro name="wheel_link" params="prefix x_location y_location">
+        <joint name="${prefix}_wheel_joint" type="continuous">
+            <parent link="chassis" />
+            <child link="${prefix}_wheel" />
+            <origin xyz="${x_location} ${y_location} ${base_link_to_wheel_z}" rpy="-${pi/2} 0 0" />
+            <axis xyz="0 0 1" />
+        </joint>
+        <link name="${prefix}_wheel">
+            <visual>
+                <geometry><cylinder radius="${wheel_radius}" length="${wheel_width}" /></geometry>
+                <material name="blue" />
+            </visual>
+            <collision>
+                <geometry><cylinder radius="${wheel_radius}" length="${wheel_width}" /></geometry>
+            </collision>
+            <xacro:inertial_cylinder mass="0.1" radius="${wheel_radius}" length="${wheel_width}">
+                <origin xyz="0 0 0" rpy="0 0 0"/>
+            </xacro:inertial_cylinder>
+        </link>
+        <gazebo reference="${prefix}_wheel">
+            <mu1 value="0.2"/>
+            <mu2 value="0.2"/>
+        </gazebo>
+    </xacro:macro>
+    <xacro:wheel_link prefix="left_front"  x_location="${base_link_to_wheel_x+box_x/2}" y_location="${base_link_to_wheel_y+box_y/2+wheel_width/2}" />
+    <xacro:wheel_link prefix="left_rear"   x_location="${box_x/2-base_link_to_wheel_x}" y_location="${base_link_to_wheel_y+box_y/2+wheel_width/2}" />
+    <xacro:wheel_link prefix="right_front" x_location="${box_x/2+base_link_to_wheel_x}" y_location="-${base_link_to_wheel_y+box_y/2+wheel_width/2}" />
+    <xacro:wheel_link prefix="right_rear"  x_location="${box_x/2-base_link_to_wheel_x}" y_location="-${base_link_to_wheel_y+box_y/2+wheel_width/2}" />
     <joint name="LiDAR_joint" type="fixed">
         <parent link="chassis" />
@@ -126,26 +96,74 @@
     <link name="laser_frame">
         <visual>
-            <geometry>
-                <cylinder radius="0.0385" length="0.019" />
-            </geometry>
+            <geometry><cylinder radius="0.0385" length="0.019" /></geometry>
             <material name="green" />
         </visual>
+        <collision>
+            <geometry><cylinder radius="0.0385" length="0.019" /></geometry>
+        </collision>
+        <xacro:inertial_cylinder mass="0.1" radius="0.0385" length="0.019">
+            <origin xyz="0 0 0" rpy="0 0 0"/>
+        </xacro:inertial_cylinder>
     </link>
-    <!-- CAMERA_LINK -->
     <xacro:property name="camera_thickness" value="0.031" />
-    <xacro:property name="chassis_to_camera_x" value="${0.210658 + camera_plate_thickness + camera_thickness/2}" />
-    <xacro:property name="chassis_to_camera_z" value="0.0156962" />
     <joint name="camera_joint" type="fixed">
         <parent link="chassis" />
         <child link="camera_link" />
-        <origin xyz="${chassis_to_camera_x} 0 ${chassis_to_camera_z+box_z}" rpy="0 0 0" />
-    </joint>©
+        <origin xyz="${0.210658 + 0.004 + camera_thickness/2} 0 ${0.0156962+box_z}" rpy="0 0 0" />
+    </joint>
     <link name="camera_link">
         <visual>
+            <geometry><box size="${camera_thickness} 0.09 0.022" /></geometry>
+            <material name="red" />
+        </visual>
+        <collision>
             <geometry>
                 <box size="${camera_thickness} 0.09 0.022" />
             </geometry>
-            <material name="red" />
-        </visual>
+        </collision>
+        <xacro:inertial_box mass="0.05" x="${camera_thickness}" y="0.09" z="0.022">
+            <origin xyz="0 0 0" rpy="0 0 0"/>
+        </xacro:inertial_box>
     </link>
+    <gazebo>
+        <plugin name="diff_drive" filename="libgazebo_ros_diff_drive.so">
+            <left_joint>left_front_wheel_joint</left_joint>
+            <right_joint>right_front_wheel_joint</right_joint>
+            <wheel_separation>${box_y + wheel_width}</wheel_separation>
+            <wheel_diameter>${wheel_diameter}</wheel_diameter>
+            <max_wheel_torque>20</max_wheel_torque>
+            <max_wheel_acceleration>1.0</max_wheel_acceleration>
+            <odometry_frame>odom</odometry_frame>
+            <robot_base_frame>base_footprint</robot_base_frame>
+            <publish_odom>true</publish_odom>
+            <publish_odom_tf>true</publish_odom_tf>
+            <publish_wheel_tf>true</publish_wheel_tf>
+        </plugin>
+    </gazebo>
+    <gazebo reference="laser_frame">
+        <material>Gazebo/Green</material>
+        <sensor name="laser" type="ray">
+            <pose> 0 0 0 0 0 0 </pose>
+            <visualize>true</visualize>
+            <update_rate>10</update_rate>
+            <ray>
+                <scan>
+                    <horizontal>
+                        <samples>360</samples>
+                        <min_angle>-3.14</min_angle>
+                        <max_angle>3.14</max_angle>
+                    </horizontal>
+                </scan>
+                <range>
+                    <min>0.1</min>
+                    <max>12</max>
+                </range>
+            </ray>
+            <plugin name="laser_controller" filename="libgazebo_ros_ray_sensor.so">
+                <ros><argument>~/out:=scan</argument></ros>
+                <output_type>sensor_msgs/LaserScan</output_type>
+                <frame_name>laser_frame</frame_name>
+            </plugin>
+        </sensor>
+    </gazebo>
 </robot>
