Commit message: URDF 최종 수정
URDF 최종 수정

File: src/forey_demo/description/my_robot.urdf (robot description, URDF)
Before this commit: robot robot, 9 links, 8 joints
Links:
- removed link camera_link
- link chassis: mass 0.8 -> 1.0
Joints:
- removed joint camera_joint
- joint left_rear_wheel_joint: origin xyz=0.024500000000000008 0.0865 -0.00602 rpy=-1.570796326795 0 0 -> xyz=0.0245 0.0865 -0.00602 rpy=-1.570796326795 0 0
- joint right_rear_wheel_joint: origin xyz=0.024500000000000008 -0.0865 -0.00602 rpy=-1.570796326795 0 0 -> xyz=0.0245 -0.0865 -0.00602 rpy=-1.570796326795 0 0
